Commit message: style: update xacro file the 'xacro:' prefix is required for a new version of the xacro format.

File: segway_description/urdf/accessories.urdf.xacro (robot description, xacro)
@@ -28,5 +28,5 @@
     <xacro:include filename="$(find segway_description)/urdf/sensors/pgr_flea3.urdf.xacro"/>
     <xacro:include filename="$(find segway_description)/urdf/sensors/garmin_18x_lvc_gps.urdf.xacro"/>
-    <property name="M_PI" value="3.14159"/>
+    <xacro:property name="M_PI" value="3.14159"/>
     <xacro:macro name="segway_accessories">
         <!-- CH Robotics UM7 Link-->
